File: code_review/headphone_amp_left.kicad_sch (KiCad schematic)
At the start: 19 parts, among them J1 Audio_Jack_3.5mm_In, J2 Audio_Jack_3.5mm_Out, P1 Power_Conn_3pin, U1 NE5532

Commit message: fix: SKILL.md wrong-format anti-patterns; fix headphone_amp_netlist.json schema
- Added '❌ WRONG Circuit IR formats' section to SKILL.md with three real
  examples of broken schemas the LLM tends to invent:
    1. title/inline-pins/dict-nets format ("REF-PIN" string notation)
    2. nested metadata wrapper with type field and inline pins
    3. hand-written .kicad_sch (old version, fake generator, no wires)
  Each is annotated with why it fails. Clear rule: if schema validation
  fails, fix the netlist — never fall back to hand-writing .kicad_sch.
- Fixed code_review/headphone_amp_netlist.json: converted from wrong schema
  to valid CircuitIR (version/components+symbol/nets with ref+pin objects).
  new-from-netlist: 18 symbols, 12 nets.
- Added code_review/headphone_amp_left.kicad_sch (OpenClaw_Managed output)
Parts:
- removed P1: Power_Conn_3pin, symbol Connector_Generic:Conn_01x03
- C1, C2: value 100nF -> 100n
- C3, C4: value 10uF -> 10u
- C5: value 1uF -> 1u
- C6: value 22uF -> 22u
- C7: value 220uF -> 220u
- J1: value Audio_Jack_3.5mm_In -> Audio_Jack_In
- J2: value Audio_Jack_3.5mm_Out -> Audio_Jack_Out
Connections:
- net RIGHT_IN_UNUSED: no longer names the net of J1.R
- net RIGHT_OUT_UNUSED: no longer names the net of J2.R
Other:
- note removed: "OpenClaw:bind={"net_name":"0V","pin":"2","ref":"P1"}"
- note removed: "OpenClaw:bind={"net_name":"RIGHT_IN_UNUSED","pin":"R","ref":"J1"}"
- note removed: "OpenClaw:bind={"net_name":"RIGHT_OUT_UNUSED","pin":"R","ref":"J2"}"
- note removed: "OpenClaw:bind={"net_name":"VMINUS15","pin":"3","ref":"P1"}"
- note removed: "OpenClaw:bind={"net_name":"VPLUS15","pin":"1","ref":"P1"}"
