File: code_review/OpenClaw_Managed.kicad_sch (KiCad schematic)
At the start: 30 parts, among them J1 STEREO_IN, J2 STEREO_OUT, U1 NE5532, U2 NE5532

Commit message: docs: fix fabricated timestamps in memory.md; update code_review assets
17 memory.md entries corrected to match actual git commit times:
- Four 2026-05-15 entries moved to correct 2026-03-01 dates
- 2026-06-02 entry corrected to 2026-03-02 (wrong month)
- Several same-day times off by 1-3 hours adjusted
- Current session entry timestamped to actual wall-clock time

Code review assets: delete stale Audio_Headphone_Amp files; add
headphone_amp_left schematic and zip from latest pipeline run.
Parts:
- removed C15: 1u, symbol Device:C
- removed C16: 22u, symbol Device:C_Polarized
- removed C17: 220u, symbol Device:C_Polarized
- removed R11, R14, R15, R17: 100k, symbol Device:R
- removed R12: 20k, symbol Device:R
- removed R13: 10k, symbol Device:R
- removed R16: 47, symbol Device:R
- removed RV2: 10k, symbol Device:R_Potentiometer
- removed U2: NE5532, symbol Amplifier_Operational:NE5532
- added J3: +15/GND/-15, symbol Connector_Generic:Conn_01x03
- C1, C2: value 100n -> 100nF
- C3, C4: value 10u -> 10uF
- C5: value 1u -> 1uF
- C6: value 22u -> 22uF
- C7: value 220u -> 220uF
- J1: value STEREO_IN -> Audio In
- J2: value STEREO_OUT -> Headphones
Connections:
- net AFTER_R6_L: no longer names the net of R6.1
- net AFTER_R6_L: now also C1.1, C3.1, C6.1, C6.2, R2.1, R2.2, R3.1, R4.1, R5.1, U1.1, U1.2 (-), U1.3 (+), J3.3 (Pin_3); no longer C7.2
- removed net BUF_L_IN: C6.1, R4.2, R5.2, RV1.2, U1.2 (-)
- removed net FB_L_NEG: C6.2, R2.1, R2.2, R3.2, R6.2, U1.1, U1.3 (+)
- removed net GND: C1.1, C2.1, C3.1, C4.2, J1.T, J2.T, R3.1, R4.1, R5.1, R7.1, RV1.1
- net HP_L_OUT renamed 0V
- net 0V: now also C1.2, C2.2, C3.2, C5.2, C7.2, J1.T, J2.T, R1.2, R3.2, R4.2, R5.2, R6.2, R7.1, RV1.1, RV1.3, J3.2 (Pin_2)
- net HP_R_OUT: no longer names the net of J2.R
- net IN_L_AC: no longer names the net of C5.1, R1.1
- net IN_L_AC: now also J1.S; no longer RV1.3
- removed net LEFT_IN: C5.2, J1.S, R1.2
- net RIGHT_IN: no longer names the net of J1.R
- removed net VMINUS15: C1.2, C2.2, C3.2, C4.1
- new net: C2.1, C4.2, J3.1 (Pin_1)
Other:
- note added: "OpenClaw:bind={"net_name":"0V","pin":"2","ref":"C1"}"
- note added: "OpenClaw:bind={"net_name":"0V","pin":"2","ref":"C2"}"
- note added: "OpenClaw:bind={"net_name":"0V","pin":"2","ref":"C3"}"
- note added: "OpenClaw:bind={"net_name":"0V","pin":"2","ref":"J3"}"
- note added: "OpenClaw:bind={"net_name":"0V","pin":"2","ref":"R3"}"
- note added: "OpenClaw:bind={"net_name":"0V","pin":"2","ref":"R4"}"
- note added: "OpenClaw:bind={"net_name":"0V","pin":"2","ref":"R5"}"
- note added: "OpenClaw:bind={"net_name":"0V","pin":"2","ref":"R7"}"
- note added: "OpenClaw:bind={"net_name":"0V","pin":"3","ref":"RV1"}"
- note added: "OpenClaw:bind={"net_name":"0V","pin":"S","ref":"J1"}"
- note added: "OpenClaw:bind={"net_name":"0V","pin":"S","ref":"J2"}"
- note added: "OpenClaw:bind={"net_name":"AFTER_R6","pin":"1","ref":"C7"}"
- note added: "OpenClaw:bind={"net_name":"AFTER_R6","pin":"2","ref":"R6"}"
- note added: "OpenClaw:bind={"net_name":"U1A_NEG","pin":"1","ref":"R3"}"
- note added: "OpenClaw:bind={"net_name":"U1A_NEG","pin":"2","ref":"R2"}"
- note added: "OpenClaw:bind={"net_name":"U1A_NEG","pin":"2","ref":"U1"}"
- note added: "OpenClaw:bind={"net_name":"VMINUS15","pin":"3","ref":"J3"}"
- note added: "OpenClaw:bind={"net_name":"VPLUS15","pin":"1","ref":"J3"}"
- note removed: "OpenClaw:bind={"net_name":"AFTER_R6_L","pin":"1","ref":"C7"}"
- note removed: "OpenClaw:bind={"net_name":"AFTER_R6_L","pin":"2","ref":"R6"}"
- note removed: "OpenClaw:bind={"net_name":"AFTER_R6_R","pin":"1","ref":"C17"}"
- note removed: "OpenClaw:bind={"net_name":"AFTER_R6_R","pin":"2","ref":"R16"}"
- note removed: "OpenClaw:bind={"net_name":"BUF_R_IN","pin":"1","ref":"R15"}"
- note removed: "OpenClaw:bind={"net_name":"BUF_R_IN","pin":"2","ref":"C16"}"
- note removed: "OpenClaw:bind={"net_name":"BUF_R_IN","pin":"5","ref":"U2"}"
- note removed: "OpenClaw:bind={"net_name":"FB_L_NEG","pin":"1","ref":"R3"}"
- note removed: "OpenClaw:bind={"net_name":"FB_L_NEG","pin":"2","ref":"R2"}"
- note removed: "OpenClaw:bind={"net_name":"FB_L_NEG","pin":"2","ref":"U1"}"
- note removed: "OpenClaw:bind={"net_name":"FB_R_NEG","pin":"1","ref":"R13"}"
- note removed: "OpenClaw:bind={"net_name":"FB_R_NEG","pin":"2","ref":"R12"}"
- note removed: "OpenClaw:bind={"net_name":"FB_R_NEG","pin":"2","ref":"U2"}"
- note removed: "OpenClaw:bind={"net_name":"GND","pin":"1","ref":"C4"}"
- note removed: "OpenClaw:bind={"net_name":"GND","pin":"2","ref":"C1"}"
- note removed: "OpenClaw:bind={"net_name":"GND","pin":"2","ref":"C2"}"
- note removed: "OpenClaw:bind={"net_name":"GND","pin":"2","ref":"C3"}"
- note removed: "OpenClaw:bind={"net_name":"GND","pin":"2","ref":"R13"}"
- note removed: "OpenClaw:bind={"net_name":"GND","pin":"2","ref":"R14"}"
- note removed: "OpenClaw:bind={"net_name":"GND","pin":"2","ref":"R15"}"
- note removed: "OpenClaw:bind={"net_name":"GND","pin":"2","ref":"R17"}"
- note removed: "OpenClaw:bind={"net_name":"GND","pin":"2","ref":"R3"}"
- note removed: "OpenClaw:bind={"net_name":"GND","pin":"2","ref":"R4"}"
- note removed: "OpenClaw:bind={"net_name":"GND","pin":"2","ref":"R5"}"
- note removed: "OpenClaw:bind={"net_name":"GND","pin":"2","ref":"R7"}"
- note removed: "OpenClaw:bind={"net_name":"GND","pin":"3","ref":"RV1"}"
- note removed: "OpenClaw:bind={"net_name":"GND","pin":"3","ref":"RV2"}"
- note removed: "OpenClaw:bind={"net_name":"GND","pin":"S","ref":"J1"}"
- note removed: "OpenClaw:bind={"net_name":"GND","pin":"S","ref":"J2"}"
- note removed: "OpenClaw:bind={"net_name":"HP_R_OUT","pin":"1","ref":"R17"}"
- note removed: "OpenClaw:bind={"net_name":"HP_R_OUT","pin":"2","ref":"C17"}"
- note removed: "OpenClaw:bind={"net_name":"HP_R_OUT","pin":"R","ref":"J2"}"
- note removed: "OpenClaw:bind={"net_name":"IN_R_AC","pin":"1","ref":"RV2"}"
- note removed: "OpenClaw:bind={"net_name":"IN_R_AC","pin":"2","ref":"C15"}"
- note removed: "OpenClaw:bind={"net_name":"IN_R_AC","pin":"2","ref":"R11"}"
- note removed: "OpenClaw:bind={"net_name":"OUT_R_STAGE1","pin":"1","ref":"C16"}"
- note removed: "OpenClaw:bind={"net_name":"OUT_R_STAGE1","pin":"1","ref":"R12"}"
- note removed: "OpenClaw:bind={"net_name":"OUT_R_STAGE1","pin":"1","ref":"U2"}"
- note removed: "OpenClaw:bind={"net_name":"OUT_R_STAGE2_RAW","pin":"1","ref":"R16"}"
- note removed: "OpenClaw:bind={"net_name":"OUT_R_STAGE2_RAW","pin":"6","ref":"U2"}"
- note removed: "OpenClaw:bind={"net_name":"OUT_R_STAGE2_RAW","pin":"7","ref":"U2"}"
- note removed: "OpenClaw:bind={"net_name":"RIGHT_IN","pin":"1","ref":"C15"}"
- note removed: "OpenClaw:bind={"net_name":"RIGHT_IN","pin":"1","ref":"R11"}"
- note removed: "OpenClaw:bind={"net_name":"RIGHT_IN","pin":"R","ref":"J1"}"
- note removed: "OpenClaw:bind={"net_name":"VMINUS15","pin":"4","ref":"U2"}"
- note removed: "OpenClaw:bind={"net_name":"VOL_R_OUT","pin":"1","ref":"R14"}"
- note removed: "OpenClaw:bind={"net_name":"VOL_R_OUT","pin":"2","ref":"RV2"}"
- note removed: "OpenClaw:bind={"net_name":"VOL_R_OUT","pin":"3","ref":"U2"}"
- note removed: "OpenClaw:bind={"net_name":"VPLUS15","pin":"8","ref":"U2"}"

Commit message: chore(code_review): update sample schematics (ne5532 rename + zip)
Parts:
- removed J3: +15/GND/-15, symbol Connector_Generic:Conn_01x03
- C1, C2: value 100nF -> 100n
- C3, C4: value 10uF -> 10u
- C5: value 1uF -> 1u
- C6: value 22uF -> 22u
- C7: value 220uF -> 220u
- J1: value Audio In -> Line In (TRS)
- J2: value Headphones -> Headphone Out (TRS)
- RV1: value 10k -> 10k log
Connections:
- net 0V: now also C1.1, C2.1, C3.1, C4.1, C4.2, C5.1, C6.1, C6.2, R1.1, R2.1, R2.2, R3.1, R4.1, R5.1, R6.1, U1.1, U1.2 (-), U1.3 (+); no longer C5.2, C7.1, C7.2, J2.S, R1.2, R6.2, R7.1
- new net: C5.2, J1.S, R1.2
- new net: C7.1, J2.S, R7.1
- new net AFTER_R6: C7.2, R6.2
Other:
- note added: "OpenClaw:bind={"net_name":"0V","pin":"1","ref":"C4"}"
- note removed: "OpenClaw:bind={"net_name":"0V","pin":"2","ref":"J3"}"
- note removed: "OpenClaw:bind={"net_name":"VMINUS15","pin":"3","ref":"J3"}"
- note removed: "OpenClaw:bind={"net_name":"VPLUS15","pin":"1","ref":"J3"}"
