File: code_review/OpAmp_Headphone_Amp_v3/OpenClaw_Managed.kicad_sch (KiCad schematic)
At the start: 18 parts, among them J1 3.5mm_IN, J2 3.5mm_OUT, U1 NE5532

Commit message: chore: replace old code_review files with OpAmp_Headphone_Amp_v3 project
Parts:
- J1: value 3.5mm_IN -> AUDIO_IN
- J2: value 3.5mm_OUT -> AUDIO_OUT
Connections:
- net HP_R_OUT: now reaches J2.R
- net RIGHT_IN: now reaches J1.R
Other:
- note added: "OpenClaw:bind={"net_name":"HP_R_OUT","pin":"R","ref":"J2"}"
- note added: "OpenClaw:bind={"net_name":"RIGHT_IN","pin":"R","ref":"J1"}"
- note added: "OpenClaw:bind={"net_name":"STAGE1_NEG","pin":"1","ref":"R3"}"
- note added: "OpenClaw:bind={"net_name":"STAGE1_NEG","pin":"2","ref":"R2"}"
- note added: "OpenClaw:bind={"net_name":"STAGE1_NEG","pin":"2","ref":"U1"}"
- note removed: "OpenClaw:bind={"net_name":"U1A_MINUS_IN","pin":"1","ref":"R3"}"
- note removed: "OpenClaw:bind={"net_name":"U1A_MINUS_IN","pin":"2","ref":"R2"}"
- note removed: "OpenClaw:bind={"net_name":"U1A_MINUS_IN","pin":"2","ref":"U1"}"
